File: Power board/Power board.kicad_pcb (KiCad board)
At the start: 2 copper layers, 66 x 100 mm, 29 parts, among them J1 High1, J10 2x2_pin_bat+, J11 2x2_pin_bat-, J2 Low1, J3 High2, J4 Low2, J5 Bat+, J6 Bat-, J7 Phase, J8 2x2_pin_support1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

Commit message: Done PCB
Parts:
- added C4: C, Capacitors_SMD:C_0805, F.Cu at (59.0, 85.0)
- added C8: C, Capacitors_SMD:C_2220, F.Cu at (59.0, 80.2)
- moved R1 4.10 mm to (31.9, 146.1), turned to 180 degrees
- moved R4 4.07 mm to (86.2, 132.5), turned to 0 degrees
- moved J1 3.45 mm to (33.5, 149.1)
- moved J4 3.25 mm to (84.8, 130.0)
- moved Q1 2.95 mm to (37.0, 137.1)
- moved Q4 2.75 mm to (81.2, 142.0)
- moved R2 2.16 mm to (72.5, 132.5), turned to 0 degrees
- moved R3 1.45 mm to (45.0, 146.0), turned to 180 degrees
- moved J2 1.00 mm to (71.0, 130.0)
- moved J3 0.50 mm to (46.5, 149.0)
Routing:
- net Net-(J4-Pad1): track 0.00 -> 4.70 mm
- net Net-(J4-Pad2): track 0.00 -> 4.66 mm
- net Net-(Q4-Pad1): track 0.00 -> 3.80 mm
