File: Power board/Power board.kicad_pcb (KiCad board)
At the start: 2 copper layers, 66 x 100 mm, 24 parts, among them J1 High1, J10 2x2_pin_bat+, J11 2x2_pin_bat-, J2 Low1, J5 Bat+, J6 Bat-, J7 Phase, J8 2x2_pin_support1, J9 2x2_pin_support2, Q2 IPB017N10N5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

Commit message: Final changes
Other:
- board text added: "Power board Group 1 Spring 2019"
Changed lines of the file:
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@@
   (general
     (thickness 0.8)
-    (drawings 21)
+    (drawings 22)
     (tracks 36)
     (zones 0)
@@
   )
   (setup
-    (last_trace_width 0.75)
+    (last_trace_width 0.25)
     (user_trace_width 0.5)
     (user_trace_width 0.6)
@@
     (tags "D2PAK DDPAK TO-263 D2PAK-7 TO-263-7 SOT-427")
     (attr smd)
-    (fp_text reference U2 (at 0 -6.65 270) (layer F.SilkS)
+    (fp_text reference U2 (at 2.125 -6.65 270) (layer F.SilkS)
       (effects (font (size 1 1) (thickness 0.15)))
     )
@@
     (tags "D2PAK DDPAK TO-263 D2PAK-7 TO-263-7 SOT-427")
     (attr smd)
-    (fp_text reference U1 (at 0 -6.65 90) (layer F.SilkS)
+    (fp_text reference U1 (at 2.125 -6.65 90) (layer F.SilkS)
       (effects (font (size 1 1) (thickness 0.15)))
     )
@@
     (tags "D2PAK DDPAK TO-263 D2PAK-7 TO-263-7 SOT-427")
     (attr smd)
-    (fp_text reference Q3 (at 0 -6.65 90) (layer F.SilkS)
+    (fp_text reference Q3 (at 2 -6.65 90) (layer F.SilkS)
       (effects (font (size 1 1) (thickness 0.15)))
     )
@@
     (zone_connect 2)
     (attr smd)
-    (fp_text reference C5 (at 0 -3.5) (layer F.SilkS)
+    (fp_text reference C5 (at 5.5 0) (layer F.SilkS)
       (effects (font (size 1 1) (thickness 0.15)))
     )
@@
     (tags "D2PAK DDPAK TO-263 D2PAK-7 TO-263-7 SOT-427")
     (attr smd)
-    (fp_text reference Q2 (at 0 -6.65 270) (layer F.SilkS)
+    (fp_text reference Q2 (at 2.5 -6.65 270) (layer F.SilkS)
       (effects (font (size 1 1) (thickness 0.15)))
     )
@@
     (zone_connect 2)
     (attr smd)
-    (fp_text reference C1 (at 0 -1.5 270) (layer F.SilkS)
+    (fp_text reference C1 (at -0.7 -1.95) (layer F.SilkS)
       (effects (font (size 1 1) (thickness 0.15)))
     )
@@
     (zone_connect 2)
     (attr smd)
-    (fp_text reference C2 (at 0 -1.5 90) (layer F.SilkS)
+    (fp_text reference C2 (at -1.3 -2 180) (layer F.SilkS)
       (effects (font (size 1 1) (thickness 0.15)))
     )
@@
     (zone_connect 2)
     (attr smd)
-    (fp_text reference R5 (at 0 -1.65 270) (layer F.SilkS)
+    (fp_text reference R5 (at 2.25 0.05) (layer F.SilkS)
       (effects (font (size 1 1) (thickness 0.15)))
     )
@@
     (zone_connect 2)
     (attr smd)
-    (fp_text reference R6 (at 0 -1.65 90) (layer F.SilkS)
+    (fp_text reference R6 (at -2.25 0 180) (layer F.SilkS)
       (effects (font (size 1 1) (thickness 0.15)))
     )
@@
     (zone_connect 2)
     (attr smd)
-    (fp_text reference C6 (at 0 -1.5) (layer F.SilkS)
+    (fp_text reference C6 (at 3 0) (layer F.SilkS)
       (effects (font (size 1 1) (thickness 0.15)))
     )
@@
     (zone_connect 2)
     (attr smd)
-    (fp_text reference C7 (at 0 -1.5) (layer F.SilkS)
+    (fp_text reference C7 (at 3 0.05) (layer F.SilkS)
       (effects (font (size 1 1) (thickness 0.15)))
     )
@@
     (zone_connect 2)
     (attr smd)
-    (fp_text reference C4 (at 0 -1.5) (layer F.SilkS)
+    (fp_text reference C4 (at -3.5 0) (layer F.SilkS)
       (effects (font (size 1 1) (thickness 0.15)))
     )
@@
     (zone_connect 2)
     (attr smd)
-    (fp_text reference C8 (at 0 -3.5) (layer F.SilkS)
+    (fp_text reference C8 (at -5.5 0.25) (layer F.SilkS)
       (effects (font (size 1 1) (thickness 0.15)))
     )
@@
       (rotate (xyz 0 0 0))
     )
+  )
+  (gr_text "Power board\nGroup 1\nSpring 2019" (at 81.5 164) (layer F.SilkS)
+    (effects (font (size 2 2) (thickness 0.4)))
   )
   (gr_arc (start 26 137) (end 26 139) (angle -180) (layer Edge.Cuts) (width 1))
@@
       (pts
         (xy 26 137.5) (xy 55.5 137.5) (xy 55.5 138.5) (xy 62 138.5) (xy 62 138)
-        (xy 92 138) (xy 92 149) (xy 76.5 149) (xy 70.5 155) (xy 70.5 171)
-        (xy 47.5 171) (xy 47.5 155) (xy 41.5 149) (xy 26 149)
+        (xy 92 138) (xy 92 149) (xy 76.5 149) (xy 70.5 155) (xy 70.5 168.5)
+        (xy 68 171) (xy 50 171) (xy 47.5 168.5) (xy 47.5 155) (xy 41.5 149)
+        (xy 26 149)
       )
     )

Commit message: Gerber files made
Parts:
- added J3: Conn_01x01, Mounting_Holes:MountingHole_3.2mm_M3_DIN965_Pad, F.Cu at (42.0, 113.0)
- added J4: Conn_01x01, Mounting_Holes:MountingHole_3.2mm_M3_DIN965_Pad, F.Cu at (76.0, 95.0)
- added REF**: MountingHole_3.2mm_M3, Mounting_Holes:MountingHole_3.2mm_M3, F.Cu at (76.0, 113.0)
- added REF**: MountingHole_3.2mm_M3, Mounting_Holes:MountingHole_3.2mm_M3, F.Cu at (42.0, 95.0)
- added REF**: MountingHole_3.2mm_M3, Mounting_Holes:MountingHole_3.2mm_M3, F.Cu at (87.0, 172.0)
- added REF**: MountingHole_3.2mm_M3, Mounting_Holes:MountingHole_3.2mm_M3, F.Cu at (31.0, 172.0)
Other:
- outline, holes or cut-outs redrawn
Changed lines of the file:
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@@
   (general
     (thickness 0.8)
-    (drawings 22)
+    (drawings 16)
     (tracks 36)
     (zones 0)
-    (modules 24)
+    (modules 30)
     (nets 18)
   )
@@
     (mod_text_size 1 1)
     (mod_text_width 0.15)
-    (pad_size 4.6 0.8)
-    (pad_drill 0)
+    (pad_size 3.2 3.2)
+    (pad_drill 3.2)
     (pad_to_mask_clearance 0.051)
     (solder_mask_min_width 0.25)
@@
     (visible_elements 7FFFFFFF)
     (pcbplotparams
-      (layerselection 0x010fc_ffffffff)
-      (usegerberextensions false)
+      (layerselection 0x010a0_7fffffff)
+      (usegerberextensions true)
       (usegerberattributes false)
       (usegerberadvancedattributes false)
@@
       (outputformat 1)
       (mirror false)
-      (drillshape 1)
+      (drillshape 0)
       (scaleselection 1)
-      (outputdirectory ""))
+      (outputdirectory "../../../Power Board gerber files/"))
   )
   (net 0 "")
@@
     (add_net "Net-(J9-Pad4)")
   )
+  (module Mounting_Holes:MountingHole_3.2mm_M3 (layer F.Cu)
+    (at 76 113)
+    (descr "Mounting Hole 3.2mm, no annular, M3")
+    (tags "mounting hole 3.2mm no annular m3")
+    (attr virtual)
+    (fp_text reference REF** (at 0 -4.2) (layer F.SilkS) hide
+      (effects (font (size 1 1) (thickness 0.15)))
+    )
+    (fp_text value MountingHole_3.2mm_M3 (at 0 4.2) (layer F.Fab)
+      (effects (font (size 1 1) (thickness 0.15)))
+    )
+    (fp_text user %R (at 0.3 0) (layer F.Fab)
+      (effects (font (size 1 1) (thickness 0.15)))
+    )
+    (fp_circle (center 0 0) (end 3.2 0) (layer Cmts.User) (width 0.15))
+    (fp_circle (center 0 0) (end 3.45 0) (layer F.CrtYd) (width 0.05))
+    (pad "" np_thru_hole circle (at 0 0) (size 3.2 3.2) (drill 3.2) (layers *.Cu *.Mask)
+      (clearance 1))
+  )
+  (module Mounting_Holes:MountingHole_3.2mm_M3 (layer F.Cu)
+    (at 42 95)
+    (descr "Mounting Hole 3.2mm, no annular, M3")
+    (tags "mounting hole 3.2mm no annular m3")
+    (attr virtual)
+    (fp_text reference REF** (at 0 -4.2) (layer F.SilkS) hide
+      (effects (font (size 1 1) (thickness 0.15)))
+    )
+    (fp_text value MountingHole_3.2mm_M3 (at 0 4.2) (layer F.Fab)
+      (effects (font (size 1 1) (thickness 0.15)))
+    )
+    (fp_text user %R (at 0.3 0) (layer F.Fab)
+      (effects (font (size 1 1) (thickness 0.15)))
+    )
+    (fp_circle (center 0 0) (end 3.2 0) (layer Cmts.User) (width 0.15))
+    (fp_circle (center 0 0) (end 3.45 0) (layer F.CrtYd) (width 0.05))
+    (pad "" np_thru_hole circle (at 0 0) (size 3.2 3.2) (drill 3.2) (layers *.Cu *.Mask)
+      (clearance 1))
+  )
+  (module Mounting_Holes:MountingHole_3.2mm_M3 (layer F.Cu)
+    (at 87 172)
+    (descr "Mounting Hole 3.2mm, no annular, M3")
+    (tags "mounting hole 3.2mm no annular m3")
+    (attr virtual)
+    (fp_text reference REF** (at 0 -4.2) (layer F.SilkS) hide
+      (effects (font (size 1 1) (thickness 0.15)))
+    )
+    (fp_text value MountingHole_3.2mm_M3 (at 0 4.2) (layer F.Fab)
+      (effects (font (size 1 1) (thickness 0.15)))
+    )
+    (fp_text user %R (at 0.3 0) (layer F.Fab)
+      (effects (font (size 1 1) (thickness 0.15)))
+    )
+    (fp_circle (center 0 0) (end 3.2 0) (layer Cmts.User) (width 0.15))
+    (fp_circle (center 0 0) (end 3.45 0) (layer F.CrtYd) (width 0.05))
+    (pad 1 np_thru_hole circle (at 0 0) (size 3.2 3.2) (drill 3.2) (layers *.Cu *.Mask))
+  )
+  (module Mounting_Holes:MountingHole_3.2mm_M3 (layer F.Cu)
+    (at 31 172)
+    (descr "Mounting Hole 3.2mm, no annular, M3")
+    (tags "mounting hole 3.2mm no annular m3")
+    (attr virtual)
+    (fp_text reference REF** (at 0 -4.2) (layer F.SilkS) hide
+      (effects (font (size 1 1) (thickness 0.15)))
+    )
+    (fp_text value MountingHole_3.2mm_M3 (at 0 4.2) (layer F.Fab)
+      (effects (font (size 1 1) (thickness 0.15)))
+    )
+    (fp_text user %R (at 0.3 0) (layer F.Fab)
+      (effects (font (size 1 1) (thickness 0.15)))
+    )
+    (fp_circle (center 0 0) (end 3.2 0) (layer Cmts.User) (width 0.15))
+    (fp_circle (center 0 0) (end 3.45 0) (layer F.CrtYd) (width 0.05))
+    (pad 1 np_thru_hole circle (at 0 0) (size 3.2 3.2) (drill 3.2) (layers *.Cu *.Mask))
+  )
   (module TO_SOT_Packages_SMD:TO-263-7_TabPin4 (layer F.Cu)
     (at 83.25 139.375 270)
@@
     )
   )
+  (module Mounting_Holes:MountingHole_3.2mm_M3_DIN965_Pad (layer F.Cu)
+    (at 42 113)
+    (descr "Mounting Hole 3.2mm, M3, DIN965")
+    (tags "mounting hole 3.2mm m3 din965")
+    (attr virtual)
+    (fp_text reference J3 (at 0 -3.8) (layer F.SilkS) hide
+      (effects (font (size 1 1) (thickness 0.15)))
+    )
+    (fp_text value Conn_01x01 (at 0 3.8) (layer F.Fab)
+      (effects (font (size 1 1) (thickness 0.15)))
+    )
+    (fp_circle (center 0 0) (end 3.05 0) (layer F.CrtYd) (width 0.05))
+    (fp_circle (center 0 0) (end 2.8 0) (layer Cmts.User) (width 0.15))
+    (fp_text user %R (at 0.3 0) (layer F.Fab)
+      (effects (font (size 1 1) (thickness 0.15)))
+    )
+    (pad 1 thru_hole circle (at 0 0) (size 5.6 5.6) (drill 3.2) (layers *.Cu *.Mask)
+      (net 8 /Bat+))
+  )
+  (module Mounting_Holes:MountingHole_3.2mm_M3_DIN965_Pad (layer F.Cu)
+    (at 76 95)
+    (descr "Mounting Hole 3.2mm, M3, DIN965")
+    (tags "mounting hole 3.2mm m3 din965")
+    (attr virtual)
+    (fp_text reference J4 (at 0 -3.8) (layer F.SilkS) hide
+      (effects (font (size 1 1) (thickness 0.15)))
+    )
+    (fp_text value Conn_01x01 (at 0 3.8) (layer F.Fab)
+      (effects (font (size 1 1) (thickness 0.15)))
+    )
+    (fp_text user %R (at 0.3 0) (layer F.Fab)
+      (effects (font (size 1 1) (thickness 0.15)))
+    )
+    (fp_circle (center 0 0) (end 2.8 0) (layer Cmts.User) (width 0.15))
+    (fp_circle (center 0 0) (end 3.05 0) (layer F.CrtYd) (width 0.05))
+    (pad 1 thru_hole circle (at 0 0) (size 5.6 5.6) (drill 3.2) (layers *.Cu *.Mask)
+      (net 9 /Bat-))
+  )
   (gr_text "Power board\nGroup 1\nSpring 2019" (at 81.5 164) (layer F.SilkS)
     (effects (font (size 2 2) (thickness 0.4)))
@@
   (gr_line (start 26 139) (end 26 177) (layer Edge.Cuts) (width 0.05))
   (gr_line (start 26 77) (end 26 135) (layer Edge.Cuts) (width 0.05))
-  (gr_circle (center 87 172) (end 88.5 172) (layer Edge.Cuts) (width 0.05))
-  (gr_circle (center 31 172) (end 32.5 172) (layer Edge.Cuts) (width 0.05))
-  (gr_circle (center 42 95) (end 43.5 95) (layer Edge.Cuts) (width 0.5))
-  (gr_circle (center 76 95) (end 77.5 95) (layer Edge.Cuts) (width 0.5))
-  (gr_circle (center 42 113) (end 43.5 113) (layer Edge.Cuts) (width 0.5))
-  (gr_circle (center 76 113) (end 77.5 113) (layer Edge.Cuts) (width 0.5))
   (gr_line (start 92 87) (end 26 87) (layer F.SilkS) (width 0.12))
   (gr_line (start 92 103) (end 26 103) (layer F.SilkS) (width 0.12))
