File: Power board/Power board.sch (KiCad schematic (older format))
At the start: 29 parts, among them J1 High1, J10 2x2_pin_bat+, J11 2x2_pin_bat-, J2 Low1, J3 High2, J4 Low2, J5 Bat+, J6 Bat-, J7 Phase, J8 2x2_pin_support1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

Commit message: Updated
Parts:
- removed J3: High2, Pin_Headers:Pin_Header_Straight_1x02_Pitch2.54mm_SMD_Pin1Left, symbol Connector_Generic:Conn_01x02
- removed J4: Low2, Pin_Headers:Pin_Header_Straight_1x02_Pitch2.54mm_SMD_Pin1Left, symbol Connector_Generic:Conn_01x02
- removed Q1, Q4: IPB017N10N5, TO_SOT_Packages_SMD:TO-263-7_TabPin4, symbol Vikings_actives:IPB017N10N5
- removed R1, R2, R3, R4: 4.7, Resistors_SMD:R_0805, symbol Device:R
- added U1, U2: IPB017N10N5-1, TO_SOT_Packages_SMD:TO-263-7_TabPin4, symbol Vikings_actives:IPB017N10N5-1
Connections:
- net Bat+: now also U1.4 (D)
- net Bat-: now also U2.2 (S), U2.3 (S), U2.5 (S), U2.6 (S)
- net at J1.1 (Pin_1): now also Q3.2 (DS), U1.7 (DS)
- net at J7.1 (Pin_1), Q2.4 (D), Q3.3 (S)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: now also U1.2 (S), U1.3 (S), U1.5 (S), U1.6 (S), U2.4 (D)
- net at Q3.1 (G): now also J1.2 (Pin_2), U1.1 (G)
- net at Q2.1 (G): now also J2.2 (Pin_2), U2.1 (G)
- net at J2.1 (Pin_1), Q2.2 (DS): now also U2.7 (DS)
Changed lines of the file:
@@
 $EndDescr
-$Comp
-L Vikings_actives:IPB017N10N5 Q1
-U 1 1 5CB8B14E
-P 4400 2250
-F 0 "Q1" H 4606 2296 50  0000 L CNN
-F 1 "IPB017N10N5" H 4606 2205 50  0000 L CNN
-F 2 "TO_SOT_Packages_SMD:TO-263-7_TabPin4" H 4400 2250 50  0001 C CIN
-F 3 "https://www.wolfspeed.com/media/downloads/145/C3M0065090J.pdf" H 4400 2250 50  0001 L CNN
-	1    4400 2250
-	1    0    0    -1
-$EndComp
 $Comp
 L Vikings_actives:IPB017N10N5 Q3
@@
 	1    0    0    -1
 $EndComp
-$Comp
-L Vikings_actives:IPB017N10N5 Q4
-U 1 1 5CB94E76
-P 6350 3250
-F 0 "Q4" H 6556 3296 50  0000 L CNN
-F 1 "IPB017N10N5" H 6556 3205 50  0000 L CNN
-F 2 "TO_SOT_Packages_SMD:TO-263-7_TabPin4" H 6350 3250 50  0001 C CIN
-F 3 "https://www.wolfspeed.com/media/downloads/145/C3M0065090J.pdf" H 6350 3250 50  0001 L CNN
-	1    6350 3250
-	1    0    0    -1
-$EndComp
 Wire Wire Line
 	4500 1700 4500 2050
@@
 Wire Wire Line
 	4500 3800 4500 3450
-$Comp
-L Device:R R1
-U 1 1 5CC099DA
-P 3900 2250
-F 0 "R1" V 3693 2250 50  0000 C CNN
-F 1 "4.7" V 3784 2250 50  0000 C CNN
-F 2 "Resistors_SMD:R_0805" V 3830 2250 50  0001 C CNN
-F 3 "~" H 3900 2250 50  0001 C CNN
-	1    3900 2250
-	0    1    1    0
-$EndComp
-$Comp
-L Device:R R2
-U 1 1 5CC0B578
-P 3900 3250
-F 0 "R2" V 3693 3250 50  0000 C CNN
-F 1 "4.7" V 3784 3250 50  0000 C CNN
-F 2 "Resistors_SMD:R_0805" V 3830 3250 50  0001 C CNN
-F 3 "~" H 3900 3250 50  0001 C CNN
-	1    3900 3250
-	0    1    1    0
-$EndComp
-$Comp
-L Device:R R4
-U 1 1 5CC0C047
-P 5850 3250
-F 0 "R4" V 5643 3250 50  0000 C CNN
-F 1 "4.7" V 5734 3250 50  0000 C CNN
-F 2 "Resistors_SMD:R_0805" V 5780 3250 50  0001 C CNN
-F 3 "~" H 5850 3250 50  0001 C CNN
-	1    5850 3250
-	0    1    1    0
-$EndComp
-$Comp
-L Device:R R3
-U 1 1 5CC100FA
-P 5850 2250
-F 0 "R3" V 5643 2250 50  0000 C CNN
-F 1 "4.7" V 5734 2250 50  0000 C CNN
-F 2 "Resistors_SMD:R_0805" V 5780 2250 50  0001 C CNN
-F 3 "~" H 5850 2250 50  0001 C CNN
-	1    5850 2250
-	0    1    1    0
-$EndComp
 Connection ~ 6450 3800
 $Comp
@@
 	4500 2450 4500 2750
 Wire Wire Line
-	6000 2250 6150 2250
-Wire Wire Line
 	4050 2250 4200 2250
 Wire Wire Line
-	6000 3250 6150 3250
-Wire Wire Line
 	4050 3250 4200 3250
-$Comp
-L Connector_Generic:Conn_01x02 J4
-U 1 1 5CC1F15C
-P 5400 3350
-F 0 "J4" H 5318 3025 50  0000 C CNN
-F 1 "Low2" H 5318 3116 50  0000 C CNN
-F 2 "Pin_Headers:Pin_Header_Straight_1x02_Pitch2.54mm_SMD_Pin1Left" H 5400 3350 50  0001 C CNN
-F 3 "~" H 5400 3350 50  0001 C CNN
-	1    5400 3350
-	-1   0    0    1
-$EndComp
-$Comp
-L Connector_Generic:Conn_01x02 J3
-U 1 1 5CC1FE1C
-P 5400 2350
-F 0 "J3" H 5318 2025 50  0000 C CNN
-F 1 "High2" H 5318 2116 50  0000 C CNN
-F 2 "Pin_Headers:Pin_Header_Straight_1x02_Pitch2.54mm_SMD_Pin1Left" H 5400 2350 50  0001 C CNN
-F 3 "~" H 5400 2350 50  0001 C CNN
-	1    5400 2350
-	-1   0    0    1
-$EndComp
 $Comp
 L Connector_Generic:Conn_01x02 J2
@@
 $EndComp
 Wire Wire Line
-	5700 2250 5600 2250
-Wire Wire Line
-	5600 2350 6150 2350
-Wire Wire Line
-	6150 3350 5600 3350
-Wire Wire Line
-	5600 3250 5700 3250
-Wire Wire Line
-	3750 3250 3650 3250
-Wire Wire Line
-	3650 3350 4200 3350
-Wire Wire Line
-	4200 2350 3650 2350
-Wire Wire Line
-	3650 2250 3750 2250
+	3650 3350 4050 3350
+Wire Wire Line
+	4200 2350 4050 2350
 Wire Wire Line
 	4500 2750 6450 2750
@@
 Wire Wire Line
 	1600 3800 2000 3800
+Wire Wire Line
+	5450 2250 5450 1950
+Wire Wire Line
+	5450 1950 4050 1950
+Wire Wire Line
+	4050 1950 4050 2250
+Wire Wire Line
+	5450 2250 6150 2250
+Wire Wire Line
+	3650 2250 4050 2250
+Connection ~ 4050 2250
+Wire Wire Line
+	5450 2350 6150 2350
+Connection ~ 4050 2350
+Wire Wire Line
+	4050 2350 3650 2350
+Wire Wire Line
+	4050 2550 5450 2550
+Wire Wire Line
+	4050 2350 4050 2550
+Wire Wire Line
+	5450 2350 5450 2550
+Wire Wire Line
+	5450 3000 4050 3000
+Wire Wire Line
+	4050 3000 4050 3250
+Wire Wire Line
+	5450 3250 6150 3250
+Wire Wire Line
+	5450 3000 5450 3250
+Wire Wire Line
+	3650 3250 4050 3250
+Connection ~ 4050 3250
+Wire Wire Line
+	4050 3350 4050 3550
+Wire Wire Line
+	4050 3550 5450 3550
+Wire Wire Line
+	5450 3550 5450 3350
+Wire Wire Line
+	5450 3350 6150 3350
+Connection ~ 4050 3350
+Wire Wire Line
+	4050 3350 4200 3350
+$Comp
+L Vikings_actives:IPB017N10N5-1 U1
+U 1 1 5CCDC810
+P 4350 2250
+F 0 "U1" H 4606 2296 50  0000 L CNN
+F 1 "IPB017N10N5-1" H 4606 2205 50  0000 L CNN
+F 2 "TO_SOT_Packages_SMD:TO-263-7_TabPin4" H 3850 1650 50  0001 C CNN
+F 3 "" H 3850 1650 50  0001 C CNN
+	1    4350 2250
+	1    0    0    -1
+$EndComp
+$Comp
+L Vikings_actives:IPB017N10N5-1 U2
+U 1 1 5CCDE070
+P 6300 3250
+F 0 "U2" H 6556 3296 50  0000 L CNN
+F 1 "IPB017N10N5-1" H 6556 3205 50  0000 L CNN
+F 2 "TO_SOT_Packages_SMD:TO-263-7_TabPin4" H 5800 2650 50  0001 C CNN
+F 3 "" H 5800 2650 50  0001 C CNN
+	1    6300 3250
+	1    0    0    -1
+$EndComp
 $EndSCHEMATC

Commit message: Gerber files made
Parts:
- added J3, J4: Conn_01x01, Mounting_Holes:MountingHole_3.2mm_M3_DIN965_Pad, symbol Connector_Generic:Conn_01x01
Connections:
- net Bat+: now also J3.1 (Pin_1)
- net Bat-: now also J4.1 (Pin_1)
Changed lines of the file:
@@
 	2000 1700 2350 1700
 Wire Wire Line
-	1000 1700 1350 1700
+	1000 1700 1100 1700
 Wire Wire Line
-	1000 3800 1350 3800
+	1000 3800 1150 3800
 $Comp
 L Device:C C8
@@
 	1    0    0    -1
 $EndComp
+$Comp
+L Connector_Generic:Conn_01x01 J3
+U 1 1 5CD9F7BF
+P 1100 1300
+F 0 "J3" V 1064 1212 50  0000 R CNN
+F 1 "Conn_01x01" V 973 1212 50  0000 R CNN
+F 2 "Mounting_Holes:MountingHole_3.2mm_M3_DIN965_Pad" H 1100 1300 50  0001 C CNN
+F 3 "~" H 1100 1300 50  0001 C CNN
+	1    1100 1300
+	0    -1   -1   0
+$EndComp
+$Comp
+L Connector_Generic:Conn_01x01 J4
+U 1 1 5CDA0D0F
+P 1150 4200
+F 0 "J4" V 1022 4280 50  0000 L CNN
+F 1 "Conn_01x01" V 1113 4280 50  0000 L CNN
+F 2 "Mounting_Holes:MountingHole_3.2mm_M3_DIN965_Pad" H 1150 4200 50  0001 C CNN
+F 3 "~" H 1150 4200 50  0001 C CNN
+	1    1150 4200
+	0    1    1    0
+$EndComp
+Wire Wire Line
+	1100 1500 1100 1700
+Connection ~ 1100 1700
+Wire Wire Line
+	1100 1700 1350 1700
+Wire Wire Line
+	1150 3800 1150 4000
+Connection ~ 1150 3800
+Wire Wire Line
+	1150 3800 1350 3800
 $EndSCHEMATC
